File: PCB/PCB_GPIO/GPIO pins.brd (EAGLE design)
At the start: 71.9 x 62.6 mm, 6 parts

Commit message: PCB_GPIO
Routing:
- net N$6: vias 0 -> 2
Changed lines of the file:
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@@
 <contactref element="SW2" pad="P$2"/>
 <contactref element="JP1" pad="15"/>
-<wire x1="10.16" y1="11.16" x2="19.05" y2="11.16" width="1.016" layer="1"/>
-<wire x1="19.05" y1="11.16" x2="19.05" y2="16.51" width="1.016" layer="1"/>
+<wire x1="10.16" y1="11.16" x2="19.05" y2="11.16" width="1.016" layer="16"/>
+<wire x1="19.05" y1="11.16" x2="19.05" y2="16.51" width="1.016" layer="16"/>
 <wire x1="19.05" y1="16.51" x2="20.32" y2="16.51" width="1.016" layer="1"/>
-<wire x1="20.32" y1="16.51" x2="20.32" y2="25.4" width="1.016" layer="1"/>
-<wire x1="20.32" y1="25.4" x2="22.86" y2="25.4" width="1.016" layer="1"/>
-<wire x1="22.86" y1="25.4" x2="22.86" y2="29.21" width="1.016" layer="1"/>
+<wire x1="20.32" y1="16.51" x2="20.32" y2="25.4" width="1.016" layer="16"/>
+<wire x1="20.32" y1="25.4" x2="22.86" y2="25.4" width="1.016" layer="16"/>
+<wire x1="22.86" y1="25.4" x2="22.86" y2="29.21" width="1.016" layer="16"/>
+<via x="20.32" y="16.51" extent="1-16" drill="0.6" shape="square"/>
+<via x="19.05" y="16.51" extent="1-16" drill="0.6" shape="square"/>
 </signal>
 <signal name="N$8">
@@
 <wire x1="2.54" y1="35.56" x2="2.54" y2="19.05" width="1.016" layer="16"/>
 <wire x1="2.54" y1="19.05" x2="7.16" y2="19.05" width="1.016" layer="16"/>
-<wire x1="17.78" y1="19.05" x2="17.78" y2="24.13" width="1.016" layer="1"/>
-<wire x1="17.78" y1="24.13" x2="2.54" y2="24.13" width="1.016" layer="1"/>
+<wire x1="17.78" y1="19.05" x2="17.78" y2="24.13" width="1.016" layer="16"/>
+<wire x1="17.78" y1="24.13" x2="2.54" y2="24.13" width="1.016" layer="16"/>
 <wire x1="2.54" y1="19.05" x2="2.54" y2="24.13" width="0" layer="19" extent="1-16"/>
 <wire x1="7.16" y1="19.05" x2="7.16" y2="19.05" width="0" layer="19" extent="1-16"/>

Commit message: PCB GPIO Final
Parts:
- removed SW1, SW2: (no value), adafruit:PUSHBUTTON_SMD_SJ
- added P1, P2: FSMCD, switch-misc:FSMCD
Connections:
- net N$5: now also P1.P$1; no longer SW1.P$2
- net N$6: now also P2.P$4; no longer SW2.P$2
- net N$7: now also P2.P$2; no longer SW2.P$1
- net N$8: now also P1.P$3; no longer SW1.P$1
Routing:
- net N$5: track 65.4 -> 58.0 mm
- net N$6: track 30.8 -> 32.1 mm, vias 2 -> 0
- net N$7: track 67.4 -> 68.4 mm
Changed lines of the file:
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@@
 <setting verticaltext="up"/>
 </settings>
-<grid distance="2" unitdist="mm" unit="mm" style="lines" multiple="1" display="yes" altdistance="2" altunitdist="mm" altunit="mm"/>
+<grid distance="0.05" unitdist="inch" unit="inch" style="lines" multiple="1" display="no" altdistance="0.025" altunitdist="inch" altunit="inch"/>
 <layers>
 <layer number="1" name="Top" color="4" fill="1" visible="yes" active="yes"/>
@@
 <attribute name="MF" value="" x="48.26" y="13.97" size="1.778" layer="27" display="off"/>
 </element>
-<element name="SW1" library="adafruit" package="PUSHBUTTON_SMD_SJ" value="" x="10.16" y="19.05" rot="R180"/>
-<element name="SW2" library="adafruit" package="PUSHBUTTON_SMD_SJ" value="" x="10.16" y="8.16" rot="R270"/>
+<element name="P1" library="switch-misc" package="FSMCD" value="FSMCD" x="10" y="16.73" rot="R90"/>
+<element name="P2" library="switch-misc" package="FSMCD" value="FSMCD" x="6.54" y="8" rot="R90"/>
 </elements>
 <signals>
@@
 </signal>
 <signal name="N$5">
-<contactref element="SW1" pad="P$2"/>
 <contactref element="JP1" pad="12"/>
 <wire x1="17.78" y1="31.75" x2="17.78" y2="38.83" width="1.016" layer="16"/>
 <wire x1="17.78" y1="38.83" x2="0" y2="38.83" width="1.016" layer="16"/>
 <wire x1="0" y1="38.83" x2="0" y2="15.24" width="1.016" layer="16"/>
-<wire x1="0" y1="15.24" x2="13.16" y2="15.24" width="1.016" layer="16"/>
-<wire x1="13.16" y1="15.24" x2="13.16" y2="19.05" width="1.016" layer="16"/>
-<wire x1="13.16" y1="19.05" x2="13.16" y2="19.05" width="0" layer="19" extent="1-16"/>
+<wire x1="0" y1="15.24" x2="3.16" y2="15.24" width="1.016" layer="16"/>
+<wire x1="3.16" y1="15.24" x2="1.16" y2="15.05" width="1.016" layer="16"/>
+<contactref element="P1" pad="P$1"/>
+<wire x1="3.16" y1="15.24" x2="6.75" y2="15.24" width="1.016" layer="16"/>
+<wire x1="6.75" y1="15.24" x2="6.75" y2="14.48" width="1.016" layer="16"/>
 </signal>
 <signal name="N$1">
@@
 </signal>
 <signal name="N$6">
-<contactref element="SW2" pad="P$2"/>
 <contactref element="JP1" pad="15"/>
-<wire x1="10.16" y1="11.16" x2="19.05" y2="11.16" width="1.016" layer="16"/>
+<wire x1="9.69" y1="11.16" x2="19.05" y2="11.16" width="1.016" layer="16"/>
 <wire x1="19.05" y1="11.16" x2="19.05" y2="16.51" width="1.016" layer="16"/>
-<wire x1="19.05" y1="16.51" x2="20.32" y2="16.51" width="1.016" layer="1"/>
+<wire x1="19.05" y1="16.51" x2="20.32" y2="16.51" width="1.016" layer="16"/>
 <wire x1="20.32" y1="16.51" x2="20.32" y2="25.4" width="1.016" layer="16"/>
 <wire x1="20.32" y1="25.4" x2="22.86" y2="25.4" width="1.016" layer="16"/>
 <wire x1="22.86" y1="25.4" x2="22.86" y2="29.21" width="1.016" layer="16"/>
-<via x="20.32" y="16.51" extent="1-16" drill="0.6" shape="square"/>
-<via x="19.05" y="16.51" extent="1-16" drill="0.6" shape="square"/>
+<contactref element="P2" pad="P$4"/>
+<wire x1="9.69" y1="11.16" x2="9.69" y2="10.25" width="1.016" layer="16"/>
 </signal>
 <signal name="N$8">
-<contactref element="SW1" pad="P$1"/>
 <contactref element="R1" pad="1"/>
 <contactref element="JP1" pad="6"/>
@@
 <wire x1="17.78" y1="19.05" x2="17.78" y2="24.13" width="1.016" layer="16"/>
 <wire x1="17.78" y1="24.13" x2="2.54" y2="24.13" width="1.016" layer="16"/>
-<wire x1="2.54" y1="19.05" x2="2.54" y2="24.13" width="0" layer="19" extent="1-16"/>
-<wire x1="7.16" y1="19.05" x2="7.16" y2="19.05" width="0" layer="19" extent="1-16"/>
+<contactref element="P1" pad="P$3"/>
+<wire x1="2.54" y1="19.05" x2="2.54" y2="24.13" width="0" layer="19" extent="16-16"/>
+<wire x1="6.7" y1="18.98" x2="2.54" y2="19.05" width="0" layer="19" extent="16-16"/>
 </signal>
 <signal name="N$3">
@@
 </signal>
 <signal name="N$7">
-<contactref element="SW2" pad="P$1"/>
 <contactref element="SG1" pad="-"/>
 <contactref element="JP1" pad="39"/>
@@
 <wire x1="21.59" y1="5.62" x2="10.16" y2="5.62" width="1.016" layer="16"/>
 <wire x1="10.16" y1="5.62" x2="10.16" y2="5.16" width="1.016" layer="16"/>
-<wire x1="10.16" y1="5.16" x2="10.16" y2="5.16" width="0" layer="19" extent="1-16"/>
+<contactref element="P2" pad="P$2"/>
+<wire x1="10.16" y1="5.16" x2="9.74" y2="5.16" width="1.016" layer="16"/>
+<wire x1="9.74" y1="5.16" x2="9.74" y2="5.75" width="1.016" layer="16"/>
 </signal>
 </signals>
