File: PCB/PCB_GPIO/GPIO pins.sch (EAGLE design)
At the start: 6 parts

Commit message: PCB GPIO Final
Parts:
- removed SW1, SW2: (no value), adafruit:SWITCH_PUSHBUTTONSOFTTOUCHSMD_SJ
- added P1, P2: FSMCD, switch-misc:FSMCD
Connections:
- net N$5: now also P1.P; no longer SW1.P$2
- net N$6: now also P2.S@1; no longer SW2.P$2
- net N$7: now also P2.P@1; no longer SW2.P$1
- net N$8: now also P1.S; no longer SW1.P$1
Changed lines of the file:
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@@
 <part name="R1" library="adafruit" deviceset="R-US_" device="0207/5V"/>
 <part name="LED1" library="adafruit" deviceset="LED" device="5MM"/>
-<part name="SW1" library="adafruit" deviceset="SWITCH_PUSHBUTTON" device="SOFTTOUCHSMD_SJ"/>
-<part name="SW2" library="adafruit" deviceset="SWITCH_PUSHBUTTON" device="SOFTTOUCHSMD_SJ"/>
 <part name="SG1" library="buzzer" deviceset="EB2209A" device=""/>
+<part name="P1" library="switch-misc" deviceset="FSMCD" device=""/>
+<part name="P2" library="switch-misc" deviceset="FSMCD" device=""/>
 </parts>
 <sheets>
@@
 <instance part="R1" gate="G$1" x="45.72" y="55.88"/>
 <instance part="LED1" gate="G$1" x="58.42" y="55.88" rot="R90"/>
-<instance part="SW1" gate="G$1" x="22.86" y="55.88"/>
-<instance part="SW2" gate="G$1" x="17.78" y="38.1"/>
 <instance part="SG1" gate="G$1" x="50.8" y="38.1" rot="R180"/>
+<instance part="P1" gate="G$1" x="22.86" y="55.88"/>
+<instance part="P2" gate="G$1" x="17.78" y="40.64"/>
 </instances>
 <busses>
@@
 <net name="N$5" class="0">
 <segment>
-<pinref part="SW1" gate="G$1" pin="P$2"/>
-<wire x1="27.94" y1="55.88" x2="27.94" y2="48.26" width="0.1524" layer="91"/>
-<wire x1="27.94" y1="48.26" x2="2.54" y2="48.26" width="0.1524" layer="91"/>
+<wire x1="20.32" y1="48.26" x2="2.54" y2="48.26" width="0.1524" layer="91"/>
 <wire x1="2.54" y1="48.26" x2="2.54" y2="93.98" width="0.1524" layer="91"/>
 <wire x1="2.54" y1="93.98" x2="27.94" y2="93.98" width="0.1524" layer="91"/>
 <pinref part="JP1" gate="A" pin="12"/>
 <wire x1="27.94" y1="93.98" x2="27.94" y2="81.28" width="0.1524" layer="91"/>
+<pinref part="P1" gate="G$1" pin="P"/>
+<wire x1="22.86" y1="50.8" x2="20.32" y2="50.8" width="0.1524" layer="91"/>
+<wire x1="20.32" y1="50.8" x2="20.32" y2="48.26" width="0.1524" layer="91"/>
 </segment>
 </net>
@@
 <net name="N$6" class="0">
 <segment>
-<pinref part="SW2" gate="G$1" pin="P$2"/>
 <wire x1="22.86" y1="38.1" x2="30.48" y2="38.1" width="0.1524" layer="91"/>
 <pinref part="JP1" gate="A" pin="15"/>
 <wire x1="30.48" y1="38.1" x2="33.02" y2="73.66" width="0.1524" layer="91"/>
+<pinref part="P2" gate="G$1" pin="S@1"/>
+<wire x1="20.32" y1="45.72" x2="22.86" y2="45.72" width="0.1524" layer="91"/>
+<wire x1="22.86" y1="45.72" x2="22.86" y2="38.1" width="0.1524" layer="91"/>
 </segment>
 </net>
@@
 <segment>
 <wire x1="5.08" y1="91.44" x2="20.32" y2="91.44" width="0.1524" layer="91"/>
-<pinref part="SW1" gate="G$1" pin="P$1"/>
-<wire x1="17.78" y1="55.88" x2="5.08" y2="55.88" width="0.1524" layer="91"/>
 <wire x1="5.08" y1="55.88" x2="5.08" y2="91.44" width="0.1524" layer="91"/>
 <pinref part="R1" gate="G$1" pin="1"/>
@@
 <wire x1="20.32" y1="88.9" x2="20.32" y2="81.28" width="0.1524" layer="91"/>
 <wire x1="20.32" y1="91.44" x2="20.32" y2="88.9" width="0.1524" layer="91"/>
+<wire x1="5.08" y1="55.88" x2="12.7" y2="55.88" width="0.1524" layer="91"/>
+<wire x1="12.7" y1="55.88" x2="12.7" y2="60.96" width="0.1524" layer="91"/>
+<pinref part="P1" gate="G$1" pin="S"/>
+<wire x1="12.7" y1="60.96" x2="22.86" y2="60.96" width="0.1524" layer="91"/>
 </segment>
 </net>
@@
 <net name="N$7" class="0">
 <segment>
-<pinref part="SW2" gate="G$1" pin="P$1"/>
-<wire x1="12.7" y1="38.1" x2="12.7" y2="33.02" width="0.1524" layer="91"/>
 <pinref part="SG1" gate="G$1" pin="-"/>
 <wire x1="45.72" y1="40.64" x2="45.72" y2="43.18" width="0.1524" layer="91"/>
@@
 <wire x1="68.58" y1="63.5" x2="68.58" y2="68.58" width="0.1524" layer="91"/>
 <wire x1="68.58" y1="68.58" x2="63.5" y2="73.66" width="0.1524" layer="91"/>
-<wire x1="12.7" y1="33.02" x2="35.56" y2="33.02" width="0.1524" layer="91"/>
+<wire x1="22.86" y1="33.02" x2="35.56" y2="33.02" width="0.1524" layer="91"/>
 <wire x1="35.56" y1="33.02" x2="45.72" y2="43.18" width="0.1524" layer="91"/>
+<pinref part="P2" gate="G$1" pin="P@1"/>
+<wire x1="20.32" y1="35.56" x2="22.86" y2="35.56" width="0.1524" layer="91"/>
+<wire x1="22.86" y1="35.56" x2="22.86" y2="33.02" width="0.1524" layer="91"/>
 </segment>
 </net>
